Commit message: feat: added new model and geomtries to rviz urdf tutorial

File: exomy_sim/models/exomy_model/exomy_model.urdf (robot description, URDF)
Before this commit: robot exomy_model, 23 links, 22 joints
Links:
- removed link bling_link
- removed link cam_link
- removed link eyewhite_link
- removed link hat_link
- removed link head_link
- removed link pupil_left_link
- removed link pupil_right_link
- added link fl_walk_link, mass 0.056321331991458; collision mesh filename=package://urdf_tutorial/meshes/fl_walk_link.STL; visual mesh filename=package://urdf_tutorial/meshes/fl_walk_link.STL
- added link fr_walk_link, mass 0.056321331991458; collision mesh filename=package://urdf_tutorial/meshes/fr_walk_link.STL; visual mesh filename=package://urdf_tutorial/meshes/fr_walk_link.STL
- added link ml_walk_link, mass 0.056321331991458; collision mesh filename=package://urdf_tutorial/meshes/ml_walk_link.STL; visual mesh filename=package://urdf_tutorial/meshes/ml_walk_link.STL
- added link mr_walk_link, mass 0.056321331991458; collision mesh filename=package://urdf_tutorial/meshes/mr_walk_link.STL; visual mesh filename=package://urdf_tutorial/meshes/mr_walk_link.STL
- added link pan_link, mass 0.0258948755353993; collision mesh filename=package://urdf_tutorial/meshes/pan_link.STL; visual mesh filename=package://urdf_tutorial/meshes/pan_link.STL
- added link rl_walk_link, mass 0.0563213319914582; collision mesh filename=package://urdf_tutorial/meshes/rl_walk_link.STL; visual mesh filename=package://urdf_tutorial/meshes/rl_walk_link.STL
- added link rr_walk_link, mass 0.056321331991458; collision mesh filename=package://urdf_tutorial/meshes/rr_walk_link.STL; visual mesh filename=package://urdf_tutorial/meshes/rr_walk_link.STL
- added link tilt_link, mass 0.0945569295049598; collision mesh filename=package://urdf_tutorial/meshes/tilt_link.STL; visual mesh filename=package://urdf_tutorial/meshes/tilt_link.STL
- link DRV_LF_link: mass 0.0569725827075566 -> 0.0578937358655145; geometry collision cylinder length=0.05 radius=0.045; visual mesh filename=package://urdf_tutorial/meshes/fl_drive_link.STL
- link DRV_LM_link: mass 0.0569725827075566 -> 0.0578937358655144; geometry collision cylinder length=0.05 radius=0.045; visual mesh filename=package://urdf_tutorial/meshes/ml_drive_link.STL
- link DRV_LR_link: mass 0.0569725827075565 -> 0.0578937358655143; geometry collision cylinder length=0.05 radius=0.045; visual mesh filename=package://urdf_tutorial/meshes/rl_drive_link.STL
- link DRV_RF_link: mass 0.0569725827075563 -> 0.0578937358655144; geometry collision cylinder length=0.05 radius=0.045; visual mesh filename=package://urdf_tutorial/meshes/fr_drive_link.STL
- link DRV_RM_link: mass 0.0569725827075566 -> 0.0578937358655146; geometry collision cylinder length=0.05 radius=0.045; visual mesh filename=package://urdf_tutorial/meshes/mr_drive_link.STL
- link DRV_RR_link: mass 0.0569725827075564 -> 0.0578937358655146; geometry collision cylinder length=0.05 radius=0.045; visual mesh filename=package://urdf_tutorial/meshes/rr_drive_link.STL
- link LFB_link: mass 0.0924731806442644 -> 0.120262550740254; geometry visual mesh filename=package://urdf_tutorial/meshes/fl_boggie_link.STL
- link MRB_link: mass 0.108378302988404 -> 0.151224745820167; geometry visual mesh filename=package://urdf_tutorial/meshes/rear_boggie_link.STL
- link RFB_link: mass 0.0924731809037187 -> 0.120262550740254; geometry visual mesh filename=package://urdf_tutorial/meshes/fr_boggie_link.STL
- link STR_LF_link: mass 0.0711741624806841 -> 0.0753331460915503; geometry visual mesh filename=package://urdf_tutorial/meshes/fl_steer_link.STL
- link STR_LM_link: mass 0.0711731050167323 -> 0.0753331460915502; geometry visual mesh filename=package://urdf_tutorial/meshes/ml_steer_link.STL
- link STR_LR_link: mass 0.0711741624806848 -> 0.0753331460915504; geometry visual mesh filename=package://urdf_tutorial/meshes/rl_steer_link.STL
- link STR_RF_link: mass 0.0711731123513564 -> 0.0753331460915505; geometry visual mesh filename=package://urdf_tutorial/meshes/fr_steer_link.STL
- link STR_RM_link: mass 0.0711741620458433 -> 0.0753331460915504; geometry visual mesh filename=package://urdf_tutorial/meshes/mr_steer_link.STL
- link STR_RR_link: mass 0.071173105016733 -> 0.0753331460915503; geometry visual mesh filename=package://urdf_tutorial/meshes/rr_steer_link.STL
- link base_link: mass 0.461792601094851 -> 0.524696065665695; geometry visual mesh filename=package://urdf_tutorial/meshes/base_link.STL
Joints:
- removed joint bling_joint
- removed joint cam_joint
- removed joint eyewhite_joint
- removed joint hat_joint
- removed joint head_joint
- removed joint pupil_left_joint
- removed joint pupil_right_joint
- added joint fl_walk_joint: type revolute, parent LFB_link, child fl_walk_link, origin xyz=0.080725 0.00453299999999998 -0.0554 rpy=0 0 0, axis 0 0 -1, limit lower=-1.57 upper=1.57 effort=0 velocity=0
- added joint fr_walk_joint: type revolute, parent RFB_link, child fr_walk_link, origin xyz=0.080725 0.004533 0.0554 rpy=-3.1416 0 0, axis 0 0 -1, limit lower=-1.57 upper=1.57 effort=0 velocity=0
- added joint ml_walk_joint: type revolute, parent LFB_link, child ml_walk_link, origin xyz=-0.0807250000000001 0.00453300000000001 -0.0553999999999999 rpy=0 0 0, axis 0 0 -1, limit lower=-1.57 upper=1.57 effort=0 velocity=0
- added joint mr_walk_joint: type revolute, parent RFB_link, child mr_walk_link, origin xyz=-0.0807250000000038 0.00453299999999712 0.0554000000000001 rpy=-3.14159265358979 0 0, axis 0 0 -1, limit lower=-1.57 upper=1.57 effort=0 velocity=0
- added joint pan_joint: type revolute, parent base_link, child pan_link, origin xyz=0.0500000000000001 0 0.26675 rpy=-3.14159265358979 0 0, axis 0 0 1, limit lower=-1.57 upper=1.57 effort=0 velocity=0
- added joint rl_walk_joint: type revolute, parent MRB_link, child rl_walk_link, origin xyz=-0.1174 0.00452999999999998 0.10372 rpy=0 1.5707963267949 0, axis 0 0 -1, limit lower=-1.57 upper=1.57 effort=0 velocity=0
- added joint rr_walk_joint: type revolute, parent MRB_link, child rr_walk_link, origin xyz=0.1174 0.00452999999999995 0.10372 rpy=3.14159265358979 1.5707963267949 0, axis 0 0 -1, limit lower=-1.57 upper=1.57 effort=0 velocity=0
- added joint tilt_joint: type revolute, parent pan_link, child tilt_link, origin xyz=0 -0.02733 -0.01145 rpy=-1.5708 0 0, axis 0 0 1, limit lower=-1.57 upper=1.57 effort=0 velocity=0
- joint DRV_LF_joint: origin xyz=0 -0.00238620000000062 -0.05724350028868 rpy=-1.5707963267949 0 0 -> xyz=0 -0.00158619999999915 -0.0576607002886822 rpy=-1.5707963267949 0 0
- joint DRV_LM_joint: origin xyz=0 -0.00238620000000191 -0.05724350028868 rpy=-1.5707963415217 0 0 -> xyz=0 -0.00158620000000223 -0.057660700288681 rpy=-1.5707963267949 0 0
- joint DRV_LR_joint: origin xyz=0 -0.0023862 -0.057244 rpy=-1.5708 0 0 -> xyz=0 -0.0015861999999994 -0.0576607002886803 rpy=-1.5707963267949 0 0
- joint DRV_RF_joint: origin xyz=0 0.00238620000000062 -0.05724350028868 rpy=-1.5707963267949 0.015893290716378 0 -> xyz=0 0.00158620000000023 -0.0576607002886802 rpy=1.5707963267949 0 0
- joint DRV_RM_joint: origin xyz=0 0.00238620000000078 -0.05724350028868 rpy=-1.57079634175582 0.0158932907163779 0 -> xyz=0 0.00158620000000148 -0.0576607002886797 rpy=1.5707963267949 0 0
- joint DRV_RR_joint: origin xyz=0 0.00238620000000078 -0.05724350028868 rpy=-1.57079634175582 0 0 -> xyz=0 0.00158620000001947 -0.0576607002886803 rpy=1.5707963267949 0 0
- joint LFB_joint: origin xyz=0.055 0.0619999999999967 0.017 rpy=-1.5707963267949 0 0 -> xyz=0.055 0.062 0.017 rpy=1.5707963267949 0 0
- joint MRB_joint: origin xyz=-0.082 0 0.017 rpy=1.5708 0 1.5708 -> xyz=-0.082 0 0.017 rpy=1.5707963267949 0 -1.5707963267949
- joint RFB_joint: origin xyz=0.055 -0.0619999999999967 0.017 rpy=-1.5707963267949 0 0 -> xyz=0.0550000000000001 -0.062 0.017 rpy=1.5707963267949 0 0
- joint STR_LF_joint: origin xyz=0.0800000000000001 0.0154182000000003 0.041775499700002 rpy=1.5707963267949 0 0 -> xyz=0 -0.0326472591798284 -0.023084199999999 rpy=-1.5707963267949 0 0; parent LFB_link -> fl_walk_link
- joint STR_LM_joint: origin xyz=-0.0799999999649664 0.0154182000000003 0.0417754997113218 rpy=1.5707963267949 0 0 -> xyz=0 -0.0326472591798298 -0.0230842000000025 rpy=-1.5707963267949 0 0; parent LFB_link -> ml_walk_link
- joint STR_LR_joint: axis 0 0 1 -> 0 0 -1; origin xyz=0.10378 -0.015418 -0.080775 rpy=0 -1.5708 -1.5708 -> xyz=0 -0.0326472591798303 -0.0230841999999993 rpy=-1.5707963267949 0 0; parent MRB_link -> rl_walk_link
- joint STR_RF_joint: origin xyz=0.0802349319288146 0.0141448430183208 -0.0417754997113241 rpy=1.5707963267949 0 -0.015893290716378 -> xyz=0 0.0326472591798303 -0.0230842 rpy=1.5707963267949 0 0; parent RFB_link -> fr_walk_link
- joint STR_RM_joint: origin xyz=-0.0797448607263364 0.0166876624779333 -0.0417754996999998 rpy=1.5707963267949 0 -0.0158932907163782 -> xyz=0 0.0326472591798309 -0.0230842000000015 rpy=1.5707963267949 0 0; parent RFB_link -> mr_walk_link
- joint STR_RR_joint: origin xyz=-0.103779999964964 -0.0154182000000004 -0.0807754997113281 rpy=0 -1.5708 -1.5708 -> xyz=0 0.0326472591798304 -0.0230841999999994 rpy=1.5707963267949 0 0; parent MRB_link -> rr_walk_link

Commit message: fix: drive and steer directions

File: exomy_sim/models/exomy_model/exomy_model.urdf (robot description, URDF)
Before this commit: robot exomy_model, 24 links, 23 joints
Joints:
- joint DRV_RF_joint: origin xyz=0 0.00158620000000023 -0.0576607002886802 rpy=1.5707963267949 0 0 -> xyz=0 0.00158620000000023 -0.0576607002886802 rpy=-1.5707963267949 0 0
- joint DRV_RM_joint: origin xyz=0 0.00158620000000148 -0.0576607002886797 rpy=1.5707963267949 0 0 -> xyz=0 0.00158620000000148 -0.0576607002886797 rpy=-1.5707963267949 0 0
- joint DRV_RR_joint: origin xyz=0 0.00158620000001947 -0.0576607002886803 rpy=1.5707963267949 0 0 -> xyz=0 0.00158620000001947 -0.0576607002886803 rpy=-1.5707963267949 0 0
- joint STR_LR_joint: axis 0 0 -1 -> 0 0 1

Commit message: feat: updated for Gazebo sim and locked walking joints to 0deg

File: exomy_sim/models/exomy_model/exomy_model.urdf (robot description, URDF)
Before this commit: robot exomy_model, 24 links, 23 joints
Links:
- link DRV_LF_link: geometry collision cylinder length=0.05 radius=0.045; visual mesh filename=package://exomy_sim/models/exomy_model/meshes/fl_drive_link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
- link DRV_LM_link: geometry collision cylinder length=0.05 radius=0.045; visual mesh filename=package://exomy_sim/models/exomy_model/meshes/ml_drive_link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
- link DRV_LR_link: geometry collision cylinder length=0.05 radius=0.045; visual mesh filename=package://exomy_sim/models/exomy_model/meshes/rl_drive_link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
- link DRV_RF_link: geometry collision cylinder length=0.05 radius=0.045; visual mesh filename=package://exomy_sim/models/exomy_model/meshes/fr_drive_link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
- link DRV_RM_link: geometry collision cylinder length=0.05 radius=0.045; visual mesh filename=package://exomy_sim/models/exomy_model/meshes/mr_drive_link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
- link DRV_RR_link: geometry collision cylinder length=0.05 radius=0.045; visual mesh filename=package://exomy_sim/models/exomy_model/meshes/rr_drive_link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
- link LFB_link: geometry visual mesh filename=package://exomy_sim/models/exomy_model/meshes/fl_boggie_lin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
- link MRB_link: geometry visual mesh filename=package://exomy_sim/models/exomy_model/meshes/rear_boggie_l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
- link RFB_link: geometry visual mesh filename=package://exomy_sim/models/exomy_model/meshes/fr_boggie_lin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
- link STR_LF_link: geometry visual mesh filename=package://exomy_sim/models/exomy_model/meshes/fl_steer_link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
- link STR_LM_link: geometry visual mesh filename=package://exomy_sim/models/exomy_model/meshes/ml_steer_link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
- link STR_LR_link: geometry visual mesh filename=package://exomy_sim/models/exomy_model/meshes/rl_steer_link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
- link STR_RF_link: geometry visual mesh filename=package://exomy_sim/models/exomy_model/meshes/fr_steer_link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
- link STR_RM_link: geometry visual mesh filename=package://exomy_sim/models/exomy_model/meshes/mr_steer_link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
- link STR_RR_link: geometry visual mesh filename=package://exomy_sim/models/exomy_model/meshes/rr_steer_link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
- link base_link: geometry visual mesh filename=package://exomy_sim/models/exomy_model/meshes/base_link.STL
- link fl_walk_link: geometry visual mesh filename=package://exomy_sim/models/exomy_model/meshes/fl_walk_link.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
- link fr_walk_link: geometry visual mesh filename=package://exomy_sim/models/exomy_model/meshes/fr_walk_link.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
- link ml_walk_link: geometry visual mesh filename=package://exomy_sim/models/exomy_model/meshes/ml_walk_link.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
- link mr_walk_link: geometry collision mesh filename=package://exomy_sim/models/exomy_model/meshes/mr_walk_link.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; visual mesh filename=package://exomy_sim/models/exomy_model/meshes/mr_walk_link.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
- link pan_link: geometry visual mesh filename=package://exomy_sim/models/exomy_model/meshes/pan_link.STL
- link rl_walk_link: geometry visual mesh filename=package://exomy_sim/models/exomy_model/meshes/rl_walk_link.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
- link rr_walk_link: geometry collision mesh filename=package://exomy_sim/models/exomy_model/meshes/rr_walk_link.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; visual mesh filename=package://exomy_sim/models/exomy_model/meshes/rr_walk_link.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
- link tilt_link: geometry visual mesh filename=package://exomy_sim/models/exomy_model/meshes/tilt_link.STL
Joints:
- joint fl_walk_joint: limit lower=-1.57 upper=1.57 effort=0 velocity=0 -> lower=0 upper=0 effort=0 velocity=0
- joint fr_walk_joint: limit lower=-1.57 upper=1.57 effort=0 velocity=0 -> lower=0 upper=0 effort=0 velocity=0
- joint ml_walk_joint: limit lower=-1.57 upper=1.57 effort=0 velocity=0 -> lower=0 upper=0 effort=0 velocity=0
- joint mr_walk_joint: limit lower=-1.57 upper=1.57 effort=0 velocity=0 -> lower=0 upper=0 effort=0 velocity=0
- joint rl_walk_joint: limit lower=-1.57 upper=1.57 effort=0 velocity=0 -> lower=0 upper=0 effort=0 velocity=0
- joint rr_walk_joint: limit lower=-1.57 upper=1.57 effort=0 velocity=0 -> lower=0 upper=0 effort=0 velocity=0

Commit message: feat: Add PTU joint control

File: exomy_sim/models/exomy_model/exomy_model.urdf (robot description, URDF)
Before this commit: robot exomy_model, 24 links, 23 joints
Joints:
- joint pan_joint: limit lower=-1.57 upper=1.57 effort=0 velocity=0 -> lower=-1.57 upper=1.57 effort=1000 velocity=1.0
- joint tilt_joint: limit lower=-1.57 upper=1.57 effort=0 velocity=0 -> lower=-1.57 upper=1.57 effort=1000 velocity=1.0
